File: hardware/RF Throwie!.kicad_sch (KiCad schematic)
At the start: 28 parts, among them J1 PWR+UART, J2 Conn_Coaxial, J4 PROG, U1 CH32V003FxUx, U2 CMT2119A, U3 ME6118A33PG, Y2 26MHz

Commit message: Add RX->DATA and TX->CLK jumpers, add more helpful silkscreen, fix SMA connector footprint
Parts:
- added JP1, JP2: SolderJumper_2_Open, Jumper:SolderJumper-2_P1.3mm_Open_RoundedPad1.0x1.5mm, symbol Jumper:SolderJumper_2_Open
Connections:
- net CLK: now also JP2.1 (A)
- net DATA: now also JP1.1 (A)
- net RX: now also JP1.2 (B)
- net TX: now also JP2.2 (B)
Other:
- note added: "C7 for additional filtering"
- note added: "Optionally tie lines together to use as CMT2119 breakout"
- note added: "To create matching network, use https://home.sandiego.edu/~ekim/e194rfs01/jwmatcher/matcher2.html to calculate the first stage (L2+C2) and https://markimicrowave.com/technical-resources/tools/lc-filter-design-tool/ to generate the rest of the filter"
- note removed: "To create matching network, use https://home.sandiego.edu/~ekim/e194rfs01/jwmatcher/matcher2.html to calculate the first stage and https://markimicrowave.com/technical-resources/tools/lc-filter-design-tool/ to generate the rest of the filter"
Changed lines of the file:
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@@
 		)
 	)
-	(text "To create matching network,\nuse https://home.sandiego.edu/~ekim/e194rfs01/jwmatcher/matcher2.html to calculate the first stage\nand https://markimicrowave.com/technical-resources/tools/lc-filter-design-tool/ to generate the rest of the filter"
+	(text "To create matching network,\nuse https://home.sandiego.edu/~ekim/e194rfs01/jwmatcher/matcher2.html to calculate the first stage (L2+C2)\nand https://markimicrowave.com/technical-resources/tools/lc-filter-design-tool/ to generate the rest of the filter"
 		(exclude_from_sim no)
 		(at 216.662 129.794 0)
@@
 		)
 	)
+	(text "C7 for additional filtering"
+		(exclude_from_sim no)
+		(at 239.776 36.576 0)
+		(effects
+			(font
+				(size 1.27 1.27)
+			)
+		)
+	)
 	(text "Short L3 and L2 for lower cost"
 		(exclude_from_sim no)
 		(at 249.682 51.054 0)
+		(effects
+			(font
+				(size 1.27 1.27)
+			)
+		)
+	)
+	(text "Optionally tie lines together to use as CMT2119 breakout"
+		(exclude_from_sim no)
+		(at 99.568 18.542 0)
 		(effects
 			(font
@@
 	(global_label "CLK"
 		(shape input)
+		(at 95.25 30.48 180)
+		(fields_autoplaced yes)
+		(effects
+			(font
+				(size 1.27 1.27)
+			)
+			(justify right)
+		)
+		(property "Intersheetrefs" "${INTERSHEET_REFS}"
+			(at 88.6967 30.48 0)
+			(effects
+				(font
+					(size 1.27 1.27)
+				)
+				(justify right)
+				(hide yes)
+			)
+		)
+	)
+	(global_label "CLK"
+		(shape input)
 		(at 77.47 69.85 180)
 		(fields_autoplaced yes)
@@
 		)
 	)
+	(global_label "TX"
+		(shape input)
+		(at 102.87 30.48 0)
+		(fields_autoplaced yes)
+		(effects
+			(font
+				(size 1.27 1.27)
+			)
+			(justify left)
+		)
+		(property "Intersheetrefs" "${INTERSHEET_REFS}"
+			(at 108.0323 30.48 0)
+			(effects
+				(font
+					(size 1.27 1.27)
+				)
+				(justify left)
+				(hide yes)
+			)
+		)
+	)
 	(global_label "DATA"
 		(shape input)
@@
 		(property "Intersheetrefs" "${INTERSHEET_REFS}"
 			(at 103.2547 82.55 0)
+			(effects
+				(font
+					(size 1.27 1.27)
+				)
+				(justify left)
+				(hide yes)
+			)
+		)
+	)
+	(global_label "DATA"
+		(shape input)
+		(at 95.25 27.94 180)
+		(fields_autoplaced yes)
+		(effects
+			(font
+				(size 1.27 1.27)
+			)
+			(justify right)
+		)
+		(property "Intersheetrefs" "${INTERSHEET_REFS}"
+			(at 87.85 27.94 0)
+			(effects
+				(font
+					(size 1.27 1.27)
+				)
+				(justify right)
+				(hide yes)
+			)
+		)
+	)
+	(global_label "RX"
+		(shape input)
+		(at 102.87 27.94 0)
+		(fields_autoplaced yes)
+		(effects
+			(font
+				(size 1.27 1.27)
+			)
+			(justify left)
+		)
+		(property "Intersheetrefs" "${INTERSHEET_REFS}"
+			(at 108.3347 27.94 0)
 			(effects
 				(font
@@
 	)
 	(symbol
+		(lib_id "Jumper:SolderJumper_2_Open")
+		(at 99.06 30.48 0)
+		(unit 1)
+		(exclude_from_sim no)
+		(in_bom no)
+		(on_board yes)
+		(dnp no)
+		(fields_autoplaced yes)
+		(property "Reference" "JP2"
+			(at 99.06 24.13 0)
+			(effects
+				(font
+					(size 1.27 1.27)
+				)
+			)
+		)
+		(property "Value" "SolderJumper_2_Open"
+			(at 99.06 26.67 0)
+			(effects
+				(font
+					(size 1.27 1.27)
+				)
+				(hide yes)
+			)
+		)
+		(property "Footprint" "Jumper:SolderJumper-2_P1.3mm_Open_RoundedPad1.0x1.5mm"
+			(at 99.06 30.48 0)
+			(effects
+				(font
+					(size 1.27 1.27)
+				)
+				(hide yes)
+			)
+		)
+		(property "Datasheet" "~"
+			(at 99.06 30.48 0)
+			(effects
+				(font
+					(size 1.27 1.27)
+				)
+				(hide yes)
+			)
+		)
+		(property "Description" "Solder Jumper, 2-pole, open"
+			(at 99.06 30.48 0)
+			(effects
+				(font
+					(size 1.27 1.27)
+				)
+				(hide yes)
+			)
+		)
+		(pin "1"
+		)
+		(pin "2"
+		)
+		(instances
+			(project "RF Throwie!"
+				(path "/01e6dee0-4d32-4b21-b740-85fb3a4879a1"
+					(reference "JP2")
+					(unit 1)
+				)
+			)
+		)
+	)
+	(symbol
 		(lib_id "power:+3.3V")
 		(at 55.88 34.29 0)
@@
 					(unit 1)
 				)
+			)
+		)
+	)
+	(symbol
+		(lib_id "Jumper:SolderJumper_2_Open")
+		(at 99.06 27.94 0)
+		(unit 1)
+		(exclude_from_sim no)
+		(in_bom no)
+		(on_board yes)
+		(dnp no)
+		(fields_autoplaced yes)
+		(property "Reference" "JP1"
+			(at 99.06 21.59 0)
+			(effects
+				(font
+					(size 1.27 1.27)
+				)
+			)
+		)
+		(property "Value" "SolderJumper_2_Open"
+			(at 99.06 24.13 0)
+			(effects
+				(font
+					(size 1.27 1.27)
+				)
+				(hide yes)
+			)
+		)
+		(property "Footprint" "Jumper:SolderJumper-2_P1.3mm_Open_RoundedPad1.0x1.5mm"
+			(at 99.06 27.94 0)
+			(effects
+				(font
+					(size 1.27 1.27)
+				)
+				(hide yes)
+			)
+		)
+		(property "Datasheet" "~"
+			(at 99.06 27.94 0)
+			(effects
+				(font
+					(size 1.27 1.27)
+				)
+				(hide yes)
+			)
+		)
+		(property "Description" "Solder Jumper, 2-pole, open"
+			(at 99.06 27.94 0)
+			(effects
+				(font
+					(size 1.27 1.27)
+				)
+				(hide yes)
+			)
+		)
+		(pin "1"
+		)
+		(pin "2"
+		)
+		(instances
+			(project ""
+				(path "/01e6dee0-4d32-4b21-b740-85fb3a4879a1"
+					(reference "JP1")
+					(unit 1)
+				)
