File: hardware/RF Throwie!.kicad_sch (KiCad schematic)
At the start: 30 parts, among them J1 PWR+UART, J2 Conn_Coaxial, J4 PROG, U1 CH32V003FxUx, U2 CMT2119A, U3 ME6118A33PG, Y2 26MHz

Commit message: First working firmware, update KiCAD, update README
Parts:
- Y2: footprint Crystal:Crystal_SMD_3225-4Pin_3.2x2.5mm -> Crystal:Crystal_SMD_2016-4Pin_2.0x1.6mm; LCSC Part Number C7294580 -> C2933002
