File: hardware/RF Throwie!.kicad_pcb (KiCad board)
At the start: 2 copper layers, 20.9 x 20.7 mm, 30 parts, among them J1 PWR+UART, J2 Conn_Coaxial, J4 PROG, U1 CH32V003FxUx, U2 CMT2119A, U3 ME6118A33PG, Y2 26MHz

Commit message: First working firmware, update KiCAD, update README
Parts:
- added REF**: MountingHole_2.2mm_M2_DIN965, MountingHole:MountingHole_2.2mm_M2_DIN965, F.Cu at (129.2, 100.7)
- Y2: footprint Crystal:Crystal_SMD_3225-4Pin_3.2x2.5mm -> Crystal:Crystal_SMD_2016-4Pin_2.0x1.6mm
- moved JP2 4.06 mm to (142.4, 98.0), turned to -90 degrees
- moved Y2 1.51 mm to (133.0, 98.9)
Routing:
- net CLK: track 12.3 -> 16.2 mm
- net TX: track 33.6 -> 35.2 mm, vias 1 -> 2
- net Net-(U2-XTAL): track 5.24 -> 4.30 mm
Other:
- outline, holes or cut-outs redrawn
- board text added: "CH32V003+CMT2119A 157-1297MHz Tx"
- board text removed: "CH32V003+CMT2119A 157-1297MHz Ultra Cheap Sub-GHz Transmitter"
